File: Kube_Module_OLED_AmbiMate/Kube-Module-OLED_AmbiMate.brd (EAGLE design)
At the start: 42.8 x 54.6 mm, 8 parts

Commit message: Added BMx280 sensor to OLED Board
Parts:
- added BMX280: (no value), con-lsta:FE06
- added SJ5: (no value), jumper:SJ_2
Connections:
- new net BMX_VCC: BMX280.6, SJ5.2
- net 3V3: now also SJ5.1
- net 5V: now also SJ5.3
- net GND: now also BMX280.5
- net SCL(D1): now also BMX280.4
- net SDA(D2): now also BMX280.3
Routing:
- net 5V: track 0.00 -> 47.4 mm
- net 3V3: track 70.7 -> 91.2 mm
- net SDA(D2): track 60.9 -> 77.1 mm
- net BMX_VCC: track 0.00 -> 8.48 mm
- net SCL(D1): track 83.0 -> 90.0 mm
Other:
- board text added: "Kube-Module-OLED_AmbiMate_v.20191221"
- board text added: "VCC"
- board text removed: "Kube-Module-OLED_AmbiMate_v.20190724"
Changed lines of the file:
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@@
 <?xml version="1.0" encoding="utf-8"?>
 <!DOCTYPE eagle SYSTEM "eagle.dtd">
-<eagle version="9.4.2">
+<eagle version="9.5.2">
 <drawing>
 <settings>
-<setting alwaysvectorfont="yes"/>
+<setting alwaysvectorfont="no"/>
 <setting verticaltext="up"/>
 </settings>
@@
 </layers>
 <board>
-<fusionsync huburn="a.cGVyc29uYWw6dWUyYjY3MDNi" projecturn="a.cGVyc29uYWw6dWUyYjY3MDNiIzIwMTcwOTEzOTI2MDQyODE" f3durn="urn:adsk.wipprod:dm.lineage:7rMSvpVYRzGI1OTpXe5Bzw" pcbguid="c67e11f8-e518-4165-89c6-4aea96db6c3c" lastpulledtime="" lastsyncedchangeguid="93ad8ff9-8277-16ac-6fee-ae68573a650f"/>
+<fusionsync huburn="a.cGVyc29uYWw6dWUyYjY3MDNi" projecturn="a.cGVyc29uYWw6dWUyYjY3MDNiIzIwMTcwOTEzOTI2MDQyODE" f3durn="urn:adsk.wipprod:dm.lineage:7rMSvpVYRzGI1OTpXe5Bzw" pcbguid="c67e11f8-e518-4165-89c6-4aea96db6c3c" lastpulledtime="" lastsyncedchangeguid="bf38705e-5f64-1972-7ae1-bca79eb005e0"/>
 <plain>
 <wire x1="16.51" y1="10.16" x2="59.36" y2="10.16" width="0" layer="20"/>
@@
 <hole x="18.2316125" y="11.720321875" drill="2"/>
 <wire x1="20.32" y1="12.7" x2="20.32" y2="27.94" width="0.1524" layer="25"/>
-<wire x1="20.32" y1="27.94" x2="55.88" y2="27.94" width="0.1524" layer="25"/>
+<wire x1="20.32" y1="27.94" x2="29.21" y2="27.94" width="0.1524" layer="25"/>
+<wire x1="29.21" y1="27.94" x2="34.29" y2="27.94" width="0.1524" layer="25"/>
+<wire x1="34.29" y1="27.94" x2="44.45" y2="27.94" width="0.1524" layer="25"/>
+<wire x1="44.45" y1="27.94" x2="55.88" y2="27.94" width="0.1524" layer="25"/>
 <wire x1="55.88" y1="27.94" x2="55.88" y2="12.7" width="0.1524" layer="25"/>
 <wire x1="55.88" y1="12.7" x2="20.32" y2="12.7" width="0.1524" layer="25"/>
-<text x="21.59" y="25.4" size="1.27" layer="25">TE AmbiMate MS4 Sensor</text>
-<text x="20.32" y="11.43" size="1.27" layer="25">Kube-Module-OLED_AmbiMate_v.20190724</text>
+<text x="25.4" y="12.7" size="1.27" layer="25">TE AmbiMate MS4 Sensor</text>
+<text x="20.32" y="11.43" size="1.27" layer="25">Kube-Module-OLED_AmbiMate_v.20191221</text>
 <text x="49.53" y="25.4" size="0.8128" layer="25">3v3</text>
 <text x="33.02" y="62.23" size="0.8128" layer="25" rot="R90">3v3</text>
@@
 <text x="20.32" y="62.23" size="0.8128" layer="25" rot="R90">5v</text>
 <text x="30.48" y="62.23" size="0.8128" layer="25" rot="R90">D4</text>
-<text x="57.15" y="11.43" size="1.27" layer="26" rot="MR0">Kube-Module-OLED_AmbiMate_v.20190724</text>
+<text x="57.15" y="11.43" size="1.27" layer="26" rot="MR0">Kube-Module-OLED_AmbiMate_v.20191221</text>
 <text x="29.21" y="49.53" size="0.8128" layer="26" rot="MR270">GND</text>
 <text x="33.02" y="49.53" size="0.8128" layer="26" rot="MR270">GND</text>
@@
 <text x="24.13" y="29.21" size="1.27" layer="25">http://www.youtube.com/c/BKHobby</text>
 <text x="53.34" y="29.21" size="1.27" layer="26" rot="MR0">http://www.youtube.com/c/BKHobby</text>
+<wire x1="29.21" y1="27.94" x2="29.21" y2="15.24" width="0.1524" layer="25"/>
+<wire x1="29.21" y1="15.24" x2="34.29" y2="15.24" width="0.1524" layer="25"/>
+<wire x1="34.29" y1="15.24" x2="44.45" y2="15.24" width="0.1524" layer="25"/>
+<wire x1="44.45" y1="15.24" x2="44.45" y2="27.94" width="0.1524" layer="25"/>
+<wire x1="34.29" y1="15.24" x2="34.29" y2="27.94" width="0.1524" layer="25"/>
+<text x="40.64" y="19.05" size="0.8128" layer="26" rot="MR270">3v3</text>
+<text x="36.83" y="19.05" size="0.8128" layer="26" rot="MR270">5v</text>
+<text x="38.1" y="25.4" size="0.8128" layer="25" rot="R270">SCL</text>
+<text x="35.56" y="25.4" size="0.8128" layer="25" rot="R270">SDA</text>
+<text x="40.64" y="25.4" size="0.8128" layer="25" rot="R270">GND</text>
+<text x="43.18" y="25.4" size="0.8128" layer="25" rot="R270">VCC</text>
 </plain>
 <attributes>
@@
 <attribute name="VALUE" x="26.75921875" y="14.013025" size="1.27" layer="27" ratio="10" rot="R90"/>
 </element>
+<element name="BMX280" library="con-lsta" library_urn="urn:adsk.eagle:library:161" package="FE06" package3d_urn="urn:adsk.eagle:package:8191/1" value="" x="36.83" y="26.67" smashed="yes">
+<attribute name="MF" value="" x="36.83" y="26.67" size="1.778" layer="27" display="off"/>
+<attribute name="MPN" value="" x="36.83" y="26.67" size="1.778" layer="27" display="off"/>
+<attribute name="NAME" x="33.02" y="19.431" size="1.27" layer="25" ratio="10"/>
+<attribute name="OC_FARNELL" value="unknown" x="36.83" y="26.67" size="1.778" layer="27" display="off"/>
+<attribute name="OC_NEWARK" value="unknown" x="36.83" y="26.67" size="1.778" layer="27" display="off"/>
+<attribute name="VALUE" x="29.21" y="23.749" size="1.27" layer="27" ratio="10"/>
+</element>
+<element name="SJ5" library="jumper" library_urn="urn:adsk.eagle:library:252" package="SJ_2" package3d_urn="urn:adsk.eagle:package:15474/1" value="" x="38.1" y="20.32" smashed="yes" rot="MR0">
+<attribute name="NAME" x="40.513" y="21.59" size="1.27" layer="26" ratio="10" rot="MR0"/>
+<attribute name="VALUE" x="38.2001" y="20.32" size="0.02" layer="28" rot="MR0"/>
+</element>
 </elements>
 <signals>
@@
 <vertex x="16.51" y="10.16"/>
 </polygon>
+<contactref element="BMX280" pad="5"/>
 </signal>
 <signal name="SCL(D1)">
@@
 <wire x1="48.006" y1="50.9016" x2="48.006" y2="50.8" width="0.1524" layer="16"/>
 <wire x1="53.34" y1="20.8788" x2="53.34" y2="20.32" width="0.1524" layer="1"/>
-<wire x1="25.4508" y1="48.768" x2="53.34" y2="20.8788" width="0.1524" layer="1"/>
+<wire x1="25.4508" y1="48.768" x2="42.3672" y2="31.8516" width="0.1524" layer="1"/>
+<wire x1="42.3672" y1="31.8516" x2="53.34" y2="20.8788" width="0.1524" layer="1"/>
 <wire x1="25.4508" y1="60.96" x2="25.4508" y2="48.768" width="0.1524" layer="1"/>
 <wire x1="25.4508" y1="60.96" x2="25.4" y2="60.96" width="0.1524" layer="1"/>
@@
 <wire x1="43.434" y1="50.9016" x2="43.434" y2="50.8" width="0.1524" layer="16"/>
 <wire x1="25.4508" y1="60.96" x2="25.4" y2="60.96" width="0.1524" layer="16"/>
+<contactref element="BMX280" pad="4"/>
+<wire x1="38.1" y1="27.5844" x2="38.1" y2="26.67" width="0.1524" layer="1"/>
+<wire x1="42.3672" y1="31.8516" x2="38.1" y2="27.5844" width="0.1524" layer="1"/>
 </signal>
 <signal name="SDA(D2)">
@@
 <wire x1="53.34" y1="23.4696" x2="53.34" y2="22.86" width="0.1524" layer="16"/>
 <wire x1="50.7492" y1="26.0604" x2="53.34" y2="23.4696" width="0.1524" layer="16"/>
-<wire x1="50.7492" y1="49.0728" x2="50.7492" y2="26.0604" width="0.1524" layer="16"/>
+<wire x1="50.7492" y1="49.0728" x2="50.7492" y2="28.6512" width="0.1524" layer="16"/>
+<wire x1="50.7492" y1="28.6512" x2="50.7492" y2="26.0604" width="0.1524" layer="16"/>
 <wire x1="50.1396" y1="49.6824" x2="50.7492" y2="49.0728" width="0.1524" layer="16"/>
 <wire x1="28.4988" y1="60.96" x2="27.94" y2="60.96" width="0.1524" layer="16"/>
@@
 <wire x1="40.386" y1="50.9016" x2="38.2524" y2="53.0352" width="0.1524" layer="16"/>
 <wire x1="40.386" y1="50.9016" x2="40.386" y2="50.8" width="0.1524" layer="16"/>
+<contactref element="BMX280" pad="3"/>
+<wire x1="35.6616" y1="27.1272" x2="35.6616" y2="26.67" width="0.1524" layer="16"/>
+<wire x1="37.1856" y1="28.6512" x2="35.6616" y2="27.1272" width="0.1524" layer="16"/>
+<wire x1="50.7492" y1="28.6512" x2="37.1856" y2="28.6512" width="0.1524" layer="16"/>
+<wire x1="35.6616" y1="26.67" x2="35.56" y2="26.67" width="0.1524" layer="16"/>
 </signal>
 <signal name="3V3">
@@
 <wire x1="33.0708" y1="60.96" x2="33.0708" y2="56.388" width="0.1524" layer="1"/>
 <wire x1="33.0708" y1="60.96" x2="33.02" y2="60.96" width="0.1524" layer="1"/>
+<contactref element="SJ5" pad="1"/>
+<wire x1="51.054" y1="20.4216" x2="39.624" y2="20.4216" width="0.1524" layer="16"/>
+<wire x1="52.2732" y1="21.6408" x2="51.054" y2="20.4216" width="0.1524" layer="16"/>
+<wire x1="54.5592" y1="21.6408" x2="52.2732" y2="21.6408" width="0.1524" layer="16"/>
+<wire x1="55.3212" y1="22.4028" x2="54.5592" y2="21.6408" width="0.1524" layer="16"/>
+<wire x1="55.3212" y1="23.3172" x2="55.3212" y2="22.4028" width="0.1524" layer="16"/>
+<wire x1="53.34" y1="25.2984" x2="55.3212" y2="23.3172" width="0.1524" layer="16"/>
+<wire x1="39.624" y1="20.4216" x2="39.624" y2="20.32" width="0.1524" layer="16"/>
+<wire x1="53.34" y1="25.2984" x2="53.34" y2="25.4" width="0.1524" layer="16"/>
 </signal>
 <signal name="5V">
 <contactref element="I2C/LED" pad="1"/>
+<contactref element="SJ5" pad="3"/>
+<wire x1="36.576" y1="23.1648" x2="36.576" y2="20.32" width="0.1524" layer="16"/>
+<wire x1="34.29" y1="25.4508" x2="36.576" y2="23.1648" width="0.1524" layer="16"/>
+<wire x1="34.29" y1="39.4716" x2="34.29" y2="25.4508" width="0.1524" layer="16"/>
+<wire x1="20.7264" y1="53.0352" x2="34.29" y2="39.4716" width="0.1524" layer="16"/>
+<wire x1="20.7264" y1="59.1312" x2="20.7264" y2="53.0352" width="0.1524" layer="16"/>
+<wire x1="20.4216" y1="59.436" x2="20.7264" y2="59.1312" width="0.1524" layer="16"/>
+<wire x1="20.4216" y1="60.96" x2="20.4216" y2="59.436" width="0.1524" layer="16"/>
+<wire x1="20.4216" y1="60.96" x2="20.32" y2="60.96" width="0.1524" layer="16"/>
 </signal>
 <signal name="LED(D4)">
 <contactref element="I2C/LED" pad="5"/>
 </signal>
+<signal name="BMX_VCC">
+<contactref element="BMX280" pad="6"/>
+<contactref element="SJ5" pad="2"/>
+<wire x1="38.1" y1="21.1836" x2="38.1" y2="20.32" width="0.1524" layer="16"/>
+<wire x1="43.1292" y1="26.2128" x2="38.1" y2="21.1836" width="0.1524" layer="16"/>
+<wire x1="43.1292" y1="26.67" x2="43.1292" y2="26.2128" width="0.1524" layer="16"/>
+<wire x1="43.1292" y1="26.67" x2="43.18" y2="26.67" width="0.1524" layer="16"/>
+</signal>
 </signals>
